File: pcb/daughterboard.kicad_pcb (KiCad board)
At the start: 2 copper layers, 22 x 31.3 mm, 51 parts, among them J1 USB_C_Receptacle_USB2.0, J2 Conn_01x02_Female, J3 Conn_01x02_Female, J4 USB_C_Receptacle_USB2.0, J5 Conn_01x02_Female, J6 Conn_01x02_Female

Commit message: reeeverse
Parts:
- FB1, FB2, J1, J4, R1, R2, R3, R4: moved to B.Cu
- moved kibuzzard-6284F97C 49.9 mm to (96.4, 62.0)
- moved kibuzzard-6284F97C 49.9 mm to (96.4, 67.3)
- moved kibuzzard-6284F97C 49.9 mm to (98.1, 88.1)
- moved kibuzzard-6284F97C 49.9 mm to (98.1, 77.7)
- moved kibuzzard-6284F97C 49.9 mm to (66.7, 77.7)
- moved kibuzzard-6284F97C 49.9 mm to (82.4, 77.7)
- moved kibuzzard-6284F97C 49.9 mm to (80.7, 62.0)
- moved kibuzzard-6284F97C 49.9 mm to (65.0, 67.3)
- moved kibuzzard-6284F97C 49.9 mm to (105.3, 64.6)
- moved kibuzzard-6284F97C 49.9 mm to (91.3, 90.7)
- moved kibuzzard-6284F97C 49.9 mm to (89.6, 64.6)
- moved kibuzzard-6284F97C 49.9 mm to (66.7, 88.1)
- moved kibuzzard-6284F97C 49.9 mm to (82.4, 88.1)
- moved kibuzzard-6284F97C 49.9 mm to (107.0, 90.7)
- moved kibuzzard-6284F97C 49.9 mm to (66.7, 82.8)
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Routing:
- net GND: track 58.4 -> 53.1 mm
- net Net-(J1-PadA7): track 14.9 -> 19.0 mm
- net Net-(J4-PadA7): track 16.1 -> 14.9 mm
- net Net-(J1-PadA6): track 13.1 -> 11.8 mm
- net Net-(J1-PadB5): track 2.62 -> 1.53 mm
- net Net-(J4-PadA5): track 2.67 -> 3.52 mm
- net Net-(J4-PadB5): track 2.17 -> 2.99 mm
- net Net-(J4-PadA4): track 14.0 -> 13.3 mm
