File: pcb/daughterboard.kicad_pcb (KiCad board)
At the start: 2 copper layers, 22 x 32.5 mm, 51 parts, among them J1 USB_C_Receptacle_USB2.0, J2 Conn_01x02_Female, J3 Conn_01x02_Female, J4 USB_C_Receptacle_USB2.0, J5 Conn_01x02_Female, J6 Conn_01x02_Female

Commit message: fix usb c
Parts:
- moved kibuzzard-6284F97C 1.31 mm to (17.4, 82.9)
- moved kibuzzard-6284F97C 1.31 mm to (19.1, 88.0)
- moved kibuzzard-6284F97C 1.31 mm to (57.7, 85.5)
- moved kibuzzard-6284F97C 1.31 mm to (28.0, 90.6)
- moved kibuzzard-6284F97C 1.31 mm to (43.6, 101.0)
- moved kibuzzard-6284F97C 1.31 mm to (59.3, 101.0)
- moved kibuzzard-6284F97C 1.31 mm to (48.8, 77.6)
- moved kibuzzard-6284F97C 1.31 mm to (48.8, 82.9)
- moved kibuzzard-6284F97C 1.31 mm to (34.7, 98.4)
- moved kibuzzard-6284F97C 1.31 mm to (43.6, 106.3)
- moved kibuzzard-6284F97C 1.31 mm to (19.0, 103.7)
- moved kibuzzard-6284F97C 1.31 mm to (50.4, 98.4)
- moved kibuzzard-6284F97C 1.31 mm to (34.7, 103.7)
- moved kibuzzard-6284F97C 1.31 mm to (59.3, 106.3)
- moved kibuzzard-6284F97C 1.31 mm to (19.0, 98.4)
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Other:
- board size 22 x 32.5 mm -> 22 x 32.8 mm
- board text added: "0.21"
- board text removed: "0.2"

Commit message: drc
Parts:
- moved kibuzzard-6284F97C 65.3 mm to (83.9, 96.5)
- moved kibuzzard-6284F97C 65.3 mm to (122.5, 94.0)
- moved kibuzzard-6284F97C 65.3 mm to (92.8, 99.1)
- moved kibuzzard-6284F97C 65.3 mm to (108.4, 109.5)
- moved kibuzzard-6284F97C 65.3 mm to (124.1, 109.5)
- moved kibuzzard-6284F97C 65.3 mm to (82.2, 91.3)
- moved kibuzzard-6284F97C 65.3 mm to (122.5, 88.7)
- moved kibuzzard-6284F97C 65.3 mm to (113.6, 86.0)
- moved kibuzzard-6284F97C 65.3 mm to (113.6, 91.3)
- moved kibuzzard-6284F97C 65.3 mm to (99.5, 106.9)
- moved kibuzzard-6284F97C 65.3 mm to (108.4, 114.8)
- moved kibuzzard-6284F97C 65.3 mm to (106.8, 88.7)
- moved kibuzzard-6284F97C 65.3 mm to (83.8, 112.2)
- moved kibuzzard-6284F97C 65.3 mm to (115.2, 106.9)
- moved kibuzzard-6284F97C 65.3 mm to (99.5, 112.2)
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Routing:
- net GND: track 30.7 -> 33.5 mm
Changed lines of the file:
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@@
   )
   (footprint "kibuzzard-6284F97C" (layer "F.Cu")
-    (at 43.64 106.32)
+    (at 108.440805 114.767041)
     (descr "Converted using: scripting")
     (tags "svg2mod")
@@
   )
   (footprint "kibuzzard-6284F97C" (layer "F.Cu")
-    (at 50.51282 93.345)
+    (at 115.313625 101.792041)
     (descr "Converted using: scripting")
     (tags "svg2mod")
@@
   )
   (footprint "kibuzzard-6284F97C" (layer "F.Cu")
-    (at 26.323555 80.202959)
+    (at 91.12436 88.65)
     (descr "Converted using: scripting")
     (tags "svg2mod")
@@
   )
   (footprint "kibuzzard-6284F97C" (layer "F.Cu")
-    (at 59.415 95.945)
+    (at 124.215805 104.392041)
     (descr "Converted using: scripting")
     (tags "svg2mod")
@@
   )
   (footprint "kibuzzard-6284F97C" (layer "F.Cu")
-    (at 33.121375 77.602959)
+    (at 97.92218 86.05)
     (descr "Converted using: scripting")
     (tags "svg2mod")
@@
   )
   (footprint "kibuzzard-6284F97C" (layer "F.Cu")
-    (at 26.321375 85.502959)
+    (at 91.12218 93.95)
     (descr "Converted using: scripting")
     (tags "svg2mod")
@@
   )
   (footprint "kibuzzard-6284F97C" (layer "F.Cu")
-    (at 59.41718 90.645)
+    (at 124.217985 99.092041)
     (descr "Converted using: scripting")
     (tags "svg2mod")
@@
   )
   (footprint "kibuzzard-6284F97C" (layer "F.Cu")
-    (at 34.815 88.045)
+    (at 99.615805 96.492041)
     (descr "Converted using: scripting")
     (tags "svg2mod")
@@
   )
   (footprint "kibuzzard-6284F97C" (layer "F.Cu")
-    (at 57.721375 85.502959)
+    (at 122.52218 93.95)
     (descr "Converted using: scripting")
     (tags "svg2mod")
@@
   )
   (footprint "kibuzzard-6284F97C" (layer "F.Cu")
-    (at 28.01718 90.645)
+    (at 92.817985 99.092041)
     (descr "Converted using: scripting")
     (tags "svg2mod")
@@
   )
   (footprint "kibuzzard-6284F97C" (layer "F.Cu")
-    (at 43.64218 101.02)
+    (at 108.442985 109.467041)
     (descr "Converted using: scripting")
     (tags "svg2mod")
@@
   )
   (footprint "kibuzzard-6284F97C" (layer "F.Cu")
-    (at 59.34218 101.02)
+    (at 124.142985 109.467041)
     (descr "Converted using: scripting")
     (tags "svg2mod")
@@
   )
   (footprint "kibuzzard-6284F97C" (layer "F.Cu")
-    (at 17.419195 82.902959)
+    (at 82.22 91.35)
     (descr "Converted using: scripting")
     (tags "svg2mod")
@@
   )
   (footprint "kibuzzard-6284F97C" (layer "F.Cu")
-    (at 57.723555 80.202959)
+    (at 122.52436 88.65)
     (descr "Converted using: scripting")
     (tags "svg2mod")
@@
   )
   (footprint "kibuzzard-6284F97C" (layer "F.Cu")
-    (at 19.115 88.045)
+    (at 83.915805 96.492041)
     (descr "Converted using: scripting")
     (tags "svg2mod")
@@
   )
   (footprint "kibuzzard-6284F97C" (layer "F.Cu")
-    (at 48.821375 77.602959)
+    (at 113.62218 86.05)
     (descr "Converted using: scripting")
     (tags "svg2mod")
@@
   )
   (footprint "kibuzzard-6284F97C" (layer "F.Cu")
-    (at 48.819195 82.902959)
+    (at 113.62 91.35)
     (descr "Converted using: scripting")
     (tags "svg2mod")
@@
   )
   (footprint "kibuzzard-6284F97C" (layer "F.Cu")
-    (at 34.74 98.42)
+    (at 99.540805 106.867041)
     (descr "Converted using: scripting")
     (tags "svg2mod")
@@
   )
   (footprint "kibuzzard-6284F97C" (layer "F.Cu")
-    (at 42.023555 80.202959)
+    (at 106.82436 88.65)
     (descr "Converted using: scripting")
     (tags "svg2mod")
@@
   )
   (footprint "kibuzzard-6284F97C" (layer "F.Cu")
-    (at 19.03782 103.72)
+    (at 83.838625 112.167041)
     (descr "Converted using: scripting")
     (tags "svg2mod")
@@
   )
   (footprint "kibuzzard-6284F97C" (layer "F.Cu")
-    (at 50.44 98.42)
+    (at 115.240805 106.867041)
     (descr "Converted using: scripting")
     (tags "svg2mod")
@@
   )
   (footprint "kibuzzard-6284F97C" (layer "F.Cu")
-    (at 34.73782 103.72)
+    (at 99.538625 112.167041)
     (descr "Converted using: scripting")
     (tags "svg2mod")
@@
   )
   (footprint "kibuzzard-6284F97C" (layer "F.Cu")
-    (at 59.34 106.32)
+    (at 124.140805 114.767041)
     (descr "Converted using: scripting")
     (tags "svg2mod")
@@
   )
   (footprint "kibuzzard-6284F97C" (layer "F.Cu")
-    (at 19.04 98.42)
+    (at 83.840805 106.867041)
     (descr "Converted using: scripting")
     (tags "svg2mod")
@@
   )
   (footprint "kibuzzard-6284F97C" (layer "F.Cu")
-    (at 27.94 106.32)
+    (at 92.740805 114.767041)
     (descr "Converted using: scripting")
     (tags "svg2mod")
@@
   )
   (footprint "kibuzzard-6284F97C" (layer "F.Cu")
-    (at 43.715 95.945)
+    (at 108.515805 104.392041)
     (descr "Converted using: scripting")
     (tags "svg2mod")
@@
   )
   (footprint "kibuzzard-6284F97C" (layer "F.Cu")
-    (at 50.43782 103.72)
+    (at 115.238625 112.167041)
     (descr "Converted using: scripting")
     (tags "svg2mod")
@@
   )
   (footprint "kibuzzard-6284F97C" (layer "F.Cu")
-    (at 43.71718 90.645)
+    (at 108.517985 99.092041)
     (descr "Converted using: scripting")
     (tags "svg2mod")
@@
   )
   (footprint "kibuzzard-6284F97C" (layer "F.Cu")
-    (at 19.11282 93.345)
+    (at 83.913625 101.792041)
     (descr "Converted using: scripting")
     (tags "svg2mod")
@@
   )
   (footprint "kibuzzard-6284F97C" (layer "F.Cu")
-    (at 27.94218 101.02)
+    (at 92.742985 109.467041)
     (descr "Converted using: scripting")
     (tags "svg2mod")
@@
   )
   (footprint "kibuzzard-6284F97C" (layer "F.Cu")
-    (at 34.81282 93.345)
+    (at 99.613625 101.792041)
     (descr "Converted using: scripting")
     (tags "svg2mod")
@@
   )
   (footprint "kibuzzard-6284F97C" (layer "F.Cu")
-    (at 42.021375 85.502959)
+    (at 106.82218 93.95)
     (descr "Converted using: scripting")
     (tags "svg2mod")
@@
   )
   (footprint "kibuzzard-6284F97C" (layer "F.Cu")
-    (at 33.119195 82.902959)
+    (at 97.92 91.35)
     (descr "Converted using: scripting")
     (tags "svg2mod")
@@
   )
   (footprint "kibuzzard-6284F97C" (layer "F.Cu")
-    (at 28.015 95.945)
+    (at 92.815805 104.392041)
     (descr "Converted using: scripting")
     (tags "svg2mod")
@@
   )
   (footprint "kibuzzard-6284F97C" (layer "F.Cu")
-    (at 50.515 88.045)
+    (at 115.315805 96.492041)
     (descr "Converted using: scripting")
     (tags "svg2mod")
@@
   )
   (footprint "kibuzzard-6284F97C" (layer "F.Cu")
-    (at 17.421375 77.602959)
+    (at 82.22218 86.05)
     (descr "Converted using: scripting")
     (tags "svg2mod")
@@
   (gr_arc (start 27.26939 88.136783) (mid 27.521483 88.16494) (end 27.76086 88.248861) (layer "Edge.Cuts") (width 0.2))
   (gr_arc (start 43.876218 88.514437) (mid 43.61439 87.799434) (end 44.244438 88.227012) (layer "Edge.Cuts") (width 0.2))
-  (gr_line (start 30.47 108.26) (end 27.47 108.26) (layer "Edge.Cuts") (width 0.1))
+  (gr_line (start 30.47 108.26) (end 27.488026 108.261974) (layer "Edge.Cuts") (width 0.1))
   (gr_arc (start 33.528302 88.238795) (mid 33.767384 88.154039) (end 34.019378 88.125002) (layer "Edge.Cuts") (width 0.2))
   (gr_line (start 30.47 102.06) (end 30.47 108.26) (layer "Edge.Cuts") (width 0.1))
@@
   )
   (segment (start 38.81 85.3) (end 40.35 85.3) (width 0.3) (layer "F.Cu") (net 1))
+  (segment (start 38.337007 101.242993) (end 39.43 100.15) (width 0.25) (layer "F.Cu") (net 1))
   (segment (start 28.627487 103.635013) (end 28.627487 101.91476) (width 0.3) (layer "F.Cu") (net 1))
+  (segment (start 38.337007 101.3625) (end 38.337007 101.242993) (width 0.25) (layer "F.Cu") (net 1))
   (segment (start 27.1 78.5375) (end 25.85 79.7875) (width 0.3) (layer "F.Cu") (net 1))
   (segment (start 25.85 79.7875) (end 25.85 83.05) (width 0.3) (layer "F.Cu") (net 1))
   (segment (start 41.15 85.4605) (end 40.5105 85.4605) (width 0.3) (layer "F.Cu") (net 1))
   (segment (start 26.534603 83.734603) (end 27.262816 83.734603) (width 0.3) (layer "F.Cu") (net 1))
+  (segment (start 39.43 100.15) (end 38.68 99.4) (width 0.25) (layer "F.Cu") (net 1))
   (segment (start 28.696124 101.846123) (end 28.696124 101.386899) (width 0.3) (layer "F.Cu") (net 1))
   (segment (start 38.15 83.1) (end 38.15 82.3375) (width 0.3) (layer "F.Cu") (net 1))
@@
   (segment (start 40.35 85.3) (end 40.5105 85.4605) (width 0.3) (layer "F.Cu") (net 1))
   (segment (start 25.85 83.05) (end 26.534603 83.734603) (width 0.3) (layer "F.Cu") (net 1))
+  (segment (start 38.68 99.4) (end 38.61 99.4) (width 0.25) (layer "F.Cu") (net 1))
   (segment (start 28.696124 101.386899) (end 27.387007 100.077782) (width 0.3) (layer "F.Cu") (net 1))
   (segment (start 27.55 104.7125) (end 28.627487 103.635013) (width 0.3) (layer "F.Cu") (net 1))
