File: pcb/daughterboard.kicad_sch (KiCad schematic)
At the start: 12 parts, among them J1 USB_C_Receptacle_USB2.0, J2 Conn_01x02_Female, J3 Conn_01x02_Female, J4 USB_C_Receptacle_USB2.0, J5 Conn_01x02_Female, J6 Conn_01x02_Female

Commit message: mid mount footprint and placement
Parts:
- J1, J4: footprint Library:C167321 -> Library:HRO-TYPE-C-31-M-13
Changed lines of the file:
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@@
     (property "Reference" "J4" (id 0) (at 106.045 30.48 0))
     (property "Value" "USB_C_Receptacle_USB2.0" (id 1) (at 106.045 33.02 0))
-    (property "Footprint" "Library:C167321" (id 2) (at 109.855 53.34 0)
+    (property "Footprint" "Library:HRO-TYPE-C-31-M-13" (id 2) (at 109.855 53.34 0)
       (effects (font (size 1.27 1.27)) hide)
     )
@@
     (property "Reference" "J1" (id 0) (at 36.195 30.48 0))
     (property "Value" "USB_C_Receptacle_USB2.0" (id 1) (at 36.195 33.02 0))
-    (property "Footprint" "Library:C167321" (id 2) (at 40.005 53.34 0)
+    (property "Footprint" "Library:HRO-TYPE-C-31-M-13" (id 2) (at 40.005 53.34 0)
       (effects (font (size 1.27 1.27)) hide)
     )
@@
     )
     (path "/f6a3288e-9575-42bb-af05-a920d59aded8"
-      (reference "J1") (unit 1) (value "USB_C_Receptacle_USB2.0") (footprint "Library:C167321")
+      (reference "J1") (unit 1) (value "USB_C_Receptacle_USB2.0") (footprint "Library:HRO-TYPE-C-31-M-13")
     )
     (path "/47993d80-a37e-426e-90c9-fd54b49ed166"
@@
     )
     (path "/dccc8a37-3fe5-4d2e-a183-bc3e80973082"
-      (reference "J4") (unit 1) (value "USB_C_Receptacle_USB2.0") (footprint "Library:C167321")
+      (reference "J4") (unit 1) (value "USB_C_Receptacle_USB2.0") (footprint "Library:HRO-TYPE-C-31-M-13")
     )
     (path "/f6222b4f-14ee-41a9-9938-9739811dada7"
